File: astra-pwr/astra-pwr.kicad_pcb (KiCad board)
At the start: 2 copper layers, 63 x 41.2 mm, 45 parts, among them J1 12V_IN, J2 RPI_PWR, J3 MISC_OUT, J4 STATUS_LED, U1 LMR54410DBVR, U2 TPS563240DDC, U3 LM321MF, U4 LM321MF, U5 LM321MF

Commit message: Finished power board
Other:
- outline, holes or cut-outs redrawn
- board text added: "ACC_UP"
- board text added: "Astra OS Power Board rev1 by Didas72"
- board text added: "BAT_LOW"
- board text added: "Carryjob: Absolem GPedrinho Silicio"
- board text added: "RPI_PWR"
